File: Drone/untitled.kicad_sch (KiCad schematic)
At the start: 0 parts

Commit message: new commit
Parts:
- added C? (x4): 4.7uF, symbol Device:C
- added C? (x2): 10uF, symbol Device:C
- added J?: Conn_01x02_Pin, symbol Connector:Conn_01x02_Pin
- added L? (x2): 2.2uH, symbol Device:L
- added R?: 4.32k, symbol Device:R
- added U? (x2): TPS62840DLCR, TPS62840DLCR:SON50P200X150X100-8N, symbol TPS62840DLCR:TPS62840DLCR
- added U?: WPME-FDSM_SIP-3, WPME-FDSM_SIP-3:WPME-FDSM_173010X78, symbol WPME-FDSM_SIP-3:WPME-FDSM_SIP-3
Connections:
- new net: L?.1, U?.7 (SW) (x2)
- new net: R?.1, U?.5 (VSET)
- new net: J?.1 (Pin_1), U?.1
- new net 1V8: C?.1, L?.2, U?.8 (VOS)
- new net 2V2: C?.1, L?.2, U?.8 (VOS)
- new net 3V3: C?.1, C?.1, U?.2 (VIN), U?.2 (VIN), U?.3
- new net Enable_Input: C?.1, C?.1, U?.4 (EN), U?.4 (EN)
- new net GND: C?.2, C?.2, C?.2, C?.2, C?.2, C?.2, J?.2 (Pin_2), R?.2, U?.1 (GND), U?.1 (GND), U?.2, U?.5 (VSET)
- new net Mode_Input: U?.3 (MODE), U?.3 (MODE)
- new net Stop_Input: U?.6 (STOP), U?.6 (STOP)
