File: Drone/Drone.kicad_sch (KiCad schematic)
At the start: 21 parts, among them IC1 STM32L412RBT6, J1 Conn_01x03_Pin, J2 USB_B_Micro, U1 ICP-10111, U2 BMI088, U3 ICU-30201

Commit message: Addded comments and connectors
Parts:
- added J3: Conn_01x06_Socket, symbol Connector:Conn_01x06_Socket
Other:
- note added: "1#ESC"
- note added: "2#ESC"
- note added: "3#ESC"
- note added: "4#ESC"
- note added: "BAT+"
- note added: "GND"
- note added: "IMU Circuit"
- note added: "Pressure Sensor"
- note added: "Ultrasonic Sensor"
Changed lines of the file:
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@@
 		(title "PCB Design Layout for Drone")
+	)
+	(text "IMU Circuit"
+		(exclude_from_sim no)
+		(at 113.284 30.988 0)
+		(effects
+			(font
+				(size 1.27 1.27)
+			)
+		)
+	)
+	(text "3#ESC"
+		(exclude_from_sim no)
+		(at 26.67 154.94 0)
+		(effects
+			(font
+				(size 1.27 1.27)
+			)
+		)
+	)
+	(text "BAT+"
+		(exclude_from_sim no)
+		(at 27.94 147.32 0)
+		(effects
+			(font
+				(size 1.27 1.27)
+			)
+		)
+	)
+	(text "4#ESC"
+		(exclude_from_sim no)
+		(at 26.67 157.226 0)
+		(effects
+			(font
+				(size 1.27 1.27)
+			)
+		)
+	)
+	(text "2#ESC"
+		(exclude_from_sim no)
+		(at 26.416 152.4 0)
+		(effects
+			(font
+				(size 1.27 1.27)
+			)
+		)
+	)
+	(text "Ultrasonic Sensor"
+		(exclude_from_sim no)
+		(at 121.92 122.174 0)
+		(effects
+			(font
+				(size 1.27 1.27)
+			)
+		)
+	)
+	(text "GND"
+		(exclude_from_sim no)
+		(at 27.432 145.034 0)
+		(effects
+			(font
+				(size 1.27 1.27)
+			)
+		)
+	)
+	(text "1#ESC"
+		(exclude_from_sim no)
+		(at 26.67 149.86 0)
+		(effects
+			(font
+				(size 1.27 1.27)
+			)
+		)
 	)
 	(text "Interrupts might be useful for the Time of Flight (ICU)"
@@
 				(bold yes)
 				(color 135 88 190 1)
+			)
+		)
+	)
+	(text "Pressure Sensor"
+		(exclude_from_sim no)
+		(at 54.864 75.184 0)
+		(effects
+			(font
+				(size 1.27 1.27)
 			)
 		)
@@
 					(unit 1)
 				)
+			)
+		)
+	)
+	(symbol
+		(lib_id "Connector:Conn_01x06_Socket")
+		(at 30.48 152.4 180)
+		(unit 1)
+		(exclude_from_sim no)
+		(in_bom yes)
+		(on_board yes)
+		(dnp no)
+		(fields_autoplaced yes)
+		(property "Reference" "J3"
+			(at 31.115 139.7 0)
+			(effects
+				(font
+					(size 1.27 1.27)
+				)
+			)
+		)
+		(property "Value" "Conn_01x06_Socket"
+			(at 31.115 142.24 0)
+			(effects
+				(font
+					(size 1.27 1.27)
+				)
+			)
+		)
+		(property "Footprint" ""
+			(at 30.48 152.4 0)
+			(effects
+				(font
+					(size 1.27 1.27)
+				)
+				(hide yes)
+			)
+		)
+		(property "Datasheet" "~"
+			(at 30.48 152.4 0)
+			(effects
+				(font
+					(size 1.27 1.27)
+				)
+				(hide yes)
+			)
+		)
+		(property "Description" "Generic connector, single row, 01x06, script generated"
+			(at 30.48 152.4 0)
+			(effects
+				(font
+					(size 1.27 1.27)
+				)
+				(hide yes)
+			)
+		)
+		(pin "2"
+		)
+		(pin "1"
+		)
+		(pin "6"
+		)
+		(pin "5"
+		)
+		(pin "4"
+		)
+		(pin "3"
+		)
+		(instances
+			(project ""
+				(path "/d78d7154-946a-48bf-8503-5b7bdc037515"
+					(reference "J3")
+					(unit 1)
+				)
